File: pixel-pump-motor-board.kicad_pcb (KiCad board)
At the start: 2 copper layers, 28.2 x 28.2 mm, 9 parts, among them J1 Conn_01x04_Female, J2 motor-connector, J3 motor-connector, Q1 STN4NF20L, U1 250X15W104MV4E

Commit message: Finished
Parts:
- added ?: , , F.Cu at (88.9, 49.9)
- added ?: , , F.Cu at (71.1, 50.0)
- added ?: , , F.Cu at (89.5, 66.7)
- added ?: , , F.Cu at (92.6, 58.5)
- added ?: , , F.Cu at (67.7, 58.7)
- added ?: , , F.Cu at (71.1, 67.3)
- added REF**: SolderWirePad_1x01_SMD_1x2mm, Connector_Wire:SolderWirePad_1x01_SMD_1x2mm, F.Cu at (80.1, 46.2)
- J1: value Conn_01x04_Female -> BM04B-SRSS-TBT(LF)(SN); footprint Connector_JST:JST_PH_B4B-PH-SM4-TB_1x04-1MP_P2.00mm_Vertical -> Connector_JST:JST_SH_BM04B-SRSS-TB_1x04-1MP_P1.00mm_Vertical
- moved C1 17.5 mm to (86.1, 51.8)
- moved J1 2.38 mm to (89.0, 58.7), turned to -90 degrees
- moved D1 0.78 mm to (85.6, 65.3), turned to 135 degrees
Routing:
- net Net-(D1-Pad2): track 0.00 -> 46.0 mm, vias 0 -> 2
- net PWM: track 0.00 -> 31.0 mm, vias 0 -> 2
- net GND: track 0.00 -> 14.1 mm, vias 0 -> 6
- net Net-(Q1-Pad1): track 0.00 -> 10.6 mm
- added copper zone on F.Cu, net +12V
- added copper zone on B.Cu, net GND

Commit message: Finish motor board
Parts:
- removed the ? at (88.9, 49.9)
- removed the ? at (71.1, 50.0)
- removed the ? at (89.5, 66.7)
- removed the ? at (92.6, 58.5)
- removed the ? at (67.7, 58.7)
- removed the ? at (71.1, 67.3)
- added ?: , , F.Cu at (89.0, 67.7)
- added ?: , , F.Cu at (67.3, 58.7)
- added ?: , , F.Cu at (80.0, 71.4)
- added ?: , , F.Cu at (92.8, 58.5)
- added ?: , , F.Cu at (88.9, 49.5)
- added ?: , , F.Cu at (70.9, 67.4)
- added ?: , , F.Cu at (71.2, 49.6)
- added D2: 2V, Diode_SMD:D_SOD-123, F.Cu at (84.0, 51.2)
- added R3: 680k, Resistor_SMD:R_0603_1608Metric, F.Cu at (85.6, 53.9)
- added R4: 120k, Resistor_SMD:R_0603_1608Metric, F.Cu at (84.7, 52.9)
- added kibuzzard-610914A4: G***, kibuzzard-610914A4, F.Cu at (71.3, 59.0)
- moved U1 17.4 mm to (85.9, 64.5), turned to -45 degrees
- moved C1 14.6 mm to (84.3, 66.3), turned to 135 degrees
- moved D1 10.1 mm to (75.5, 65.6), turned to 45 degrees
- moved J1 1.16 mm to (88.0, 59.1), turned to 90 degrees
- moved Q1 0.75 mm to (75.4, 55.3)
- moved REF** 0.21 mm to (80.2, 46.0)
Connections:
- net +12V renamed BEMF_PIN
Routing:
- net BEMF_PIN: track 0.00 -> 43.2 mm, vias 0 -> 6
- net GND: track 14.1 -> 1.65 mm, vias 6 -> 23
- net BEMF: track 0.00 -> 10.3 mm, vias 0 -> 2
- net PWM: track 31.0 -> 21.1 mm
- net Net-(D1-Pad2): track 46.0 -> 36.3 mm, vias 2 -> 5
- net Net-(Q1-Pad1): track 10.6 -> 12.5 mm, vias 0 -> 3
- added copper zone on F.Cu, net GND
- removed copper zone on F.Cu, net BEMF_PIN
Other:
- board text added: "MOTOR DRIVER"
- board text added: "Rev 1"

Commit message: Cleanup and generate iBOM
Parts:
- removed ? (x7): , 
- removed REF**: SolderWirePad_1x01_SMD_1x2mm, Connector_Wire:SolderWirePad_1x01_SMD_1x2mm
- C1: value C_Polarized -> 100n 25V
- moved J3 20.8 mm to (71.3, 55.3), turned to 0 degrees
- moved J2 0.08 mm to (71.3, 73.3)
Changed lines of the file:
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@@
     )
-  )
-  (footprint "" (layer "F.Cu")
-    (at 89.05 67.7)
-    (fp_text reference "" (at 0 0) (layer "F.SilkS")
-      (effects (font (size 1.27 1.27) (thickness 0.15)))
-    )
-    (fp_text value "" (at 0 0) (layer "F.SilkS")
-      (effects (font (size 1.27 1.27) (thickness 0.15)))
-    )
-    (pad "1" smd roundrect (at 0 0 45) (size 1 2) (layers "B.Cu" "B.Mask") (roundrect_rratio 0.25)
-      (net 2 "GND"))
   )
   (footprint "motor-mount:motor-mount" (layer "F.Cu")
-    (at 88.8816 44.0436 180)
-    (property "Sheetfile" "pixel-pump-motor-board.kicad_sch")
-    (property "Sheetname" "")
-    (fp_text reference "J3" (at 8.89 -12.168 180 unlocked) (layer "F.SilkS") hide
-      (effects (font (size 1 1) (thickness 0.15)))
-    )
-    (fp_text value "motor-connector" (at 8.89 -10.668 180 unlocked) (layer "F.Fab")
-      (effects (font (size 1 1) (thickness 0.15)))
-    )
-    (fp_text user "${REFERENCE}" (at 8.89 -9.168 180 unlocked) (layer "F.Fab")
-      (effects (font (size 1 1) (thickness 0.15)))
-    )
-    (pad "" thru_hole oval (at 8.77 -5.588 180) (size 2.6 4.2) (drill oval 1 3) (layers *.Cu "F.Mask") (remove_unused_layers)
-      (net 3 "Net-(D1-Pad2)") (pinfunction "motor"))
-  )
-  (footprint "" (layer "F.Cu")
-    (at 67.35 58.7 90)
-    (fp_text reference "" (at 0 0 90) (layer "F.SilkS")
-      (effects (font (size 1.27 1.27) (thickness 0.15)))
-    )
-    (fp_text value "" (at 0 0 90) (layer "F.SilkS")
-      (effects (font (size 1.27 1.27) (thickness 0.15)))
-    )
-    (pad "1" smd roundrect (at 0 0 90) (size 1 2) (layers "B.Cu" "B.Mask") (roundrect_rratio 0.25)
-      (net 2 "GND"))
+    (at 71.33 55.263)
+    (property "Sheetfile" "pixel-pump-motor-board.kicad_sch")
+    (property "Sheetname" "")
+    (fp_text reference "J3" (at 8.89 -12.168 unlocked) (layer "F.SilkS")
+      (effects (font (size 1 1) (thickness 0.15)))
+    )
+    (fp_text value "motor-connector" (at 8.89 -10.668 unlocked) (layer "F.Fab")
+      (effects (font (size 1 1) (thickness 0.15)))
+    )
+    (fp_text user "${REFERENCE}" (at 8.89 -9.168 unlocked) (layer "F.Fab")
+      (effects (font (size 1 1) (thickness 0.15)))
+    )
+    (pad "1" thru_hole oval (at 8.77 -5.588) (size 2.5 4.2) (drill oval 1 3) (layers *.Cu "F.Mask") (remove_unused_layers)
+      (net 3 "Net-(D1-Pad2)") (pinfunction "motor") (pintype "bidirectional"))
   )
   (footprint "kibuzzard-610914A4" (layer "F.Cu")
@@
       (effects (font (size 0.65 0.65) (thickness 0.13)))
     )
-    (fp_text value "C_Polarized" (at 0 1.75 135) (layer "F.Fab")
+    (fp_text value "100n 25V" (at 0 1.75 135) (layer "F.Fab")
       (effects (font (size 1 1) (thickness 0.15)))
     )
@@
     )
   )
-  (footprint "" (layer "F.Cu")
-    (at 79.95 71.375)
-    (fp_text reference "" (at 0 0) (layer "F.SilkS")
-      (effects (font (size 1.27 1.27) (thickness 0.15)))
-    )
-    (fp_text value "" (at 0 0) (layer "F.SilkS")
-      (effects (font (size 1.27 1.27) (thickness 0.15)))
-    )
-    (pad "1" smd roundrect (at 0 0) (size 1 2) (layers "B.Cu" "B.Mask") (roundrect_rratio 0.25)
-      (net 2 "GND"))
-  )
   (footprint "Resistor_SMD:R_0603_1608Metric" (layer "F.Cu")
     (at 73.406 63.6524 45)
@@
     )
   )
-  (footprint "" (layer "F.Cu")
-    (at 92.8 58.475 90)
-    (fp_text reference "" (at 0 0 90) (layer "F.SilkS")
-      (effects (font (size 1.27 1.27) (thickness 0.15)))
-    )
-    (fp_text value "" (at 0 0 90) (layer "F.SilkS")
-      (effects (font (size 1.27 1.27) (thickness 0.15)))
-    )
-    (pad "1" smd roundrect (at 0 0 90) (size 1 2) (layers "B.Cu" "B.Mask") (roundrect_rratio 0.25)
-      (net 2 "GND"))
-  )
   (footprint "Resistor_SMD:R_0603_1608Metric" (layer "F.Cu")
     (at 84.65 52.925 45)
@@
     )
   )
-  (footprint "" (layer "F.Cu")
-    (at 88.925 49.45 90)
-    (fp_text reference "" (at 0 0 90) (layer "F.SilkS")
-      (effects (font (size 1.27 1.27) (thickness 0.15)))
-    )
-    (fp_text value "" (at 0 0 90) (layer "F.SilkS")
-      (effects (font (size 1.27 1.27) (thickness 0.15)))
-    )
-    (pad "1" smd roundrect (at 0 0 135) (size 1 2) (layers "B.Cu" "B.Mask") (roundrect_rratio 0.25)
-      (net 2 "GND"))
-  )
-  (footprint "" (layer "F.Cu")
-    (at 70.875 67.425 90)
-    (fp_text reference "" (at 0 0 90) (layer "F.SilkS")
-      (effects (font (size 1.27 1.27) (thickness 0.15)))
-    )
-    (fp_text value "" (at 0 0 90) (layer "F.SilkS")
-      (effects (font (size 1.27 1.27) (thickness 0.15)))
-    )
-    (pad "1" smd roundrect (at 0 0 135) (size 1 2) (layers "B.Cu" "B.Mask") (roundrect_rratio 0.25)
-      (net 2 "GND"))
+  (footprint "motor-mount:motor-mount" (layer "F.Cu")
+    (at 71.255 73.263)
+    (property "Sheetfile" "pixel-pump-motor-board.kicad_sch")
+    (property "Sheetname" "")
+    (fp_text reference "J2" (at 8.89 -12.168 unlocked) (layer "F.SilkS")
+      (effects (font (size 1 1) (thickness 0.15)))
+    )
+    (fp_text value "motor-connector" (at 8.89 -10.668 unlocked) (layer "F.Fab")
+      (effects (font (size 1 1) (thickness 0.15)))
+    )
+    (fp_text user "${REFERENCE}" (at 8.89 -9.168 unlocked) (layer "F.Fab")
+      (effects (font (size 1 1) (thickness 0.15)))
+    )
+    (pad "1" thru_hole oval (at 8.77 -5.588) (size 2.5 4.2) (drill oval 1 3) (layers *.Cu "F.Mask") (remove_unused_layers)
+      (net 1 "BEMF_PIN") (pinfunction "motor") (pintype "bidirectional"))
   )
   (footprint "Resistor_SMD:R_0603_1608Metric" (layer "F.Cu")
@@
     )
   )
-  (footprint "" (layer "F.Cu")
-    (at 71.175 49.575)
-    (fp_text reference "" (at 0 0) (layer "F.SilkS")
-      (effects (font (size 1.27 1.27) (thickness 0.15)))
-    )
-    (fp_text value "" (at 0 0) (layer "F.SilkS")
-      (effects (font (size 1.27 1.27) (thickness 0.15)))
-    )
-    (pad "1" smd roundrect (at 0 0 45) (size 1 2) (layers "B.Cu" "B.Mask") (roundrect_rratio 0.25)
-      (net 2 "GND"))
-  )
   (footprint "Resistor_SMD:R_0603_1608Metric" (layer "F.Cu")
     (at 85.625 53.875 -135)
@@
       (rotate (xyz 0 0 0))
     )
-  )
-  (footprint "Connector_Wire:SolderWirePad_1x01_SMD_1x2mm" (layer "F.Cu")
-    (at 80.175 46.025)
-    (descr "Wire Pad, Square, SMD Pad,  5mm x 10mm,")
-    (tags "MesurementPoint Square SMDPad 5mmx10mm ")
-    (attr exclude_from_pos_files exclude_from_bom)
-    (fp_text reference "REF**" (at 0 -2.54) (layer "F.SilkS")
-      (effects (font (size 1 1) (thickness 0.15)))
-    )
-    (fp_text value "SolderWirePad_1x01_SMD_1x2mm" (at 0 2.54) (layer "F.Fab")
-      (effects (font (size 1 1) (thickness 0.15)))
-    )
-    (fp_text user "${REFERENCE}" (at 0 0) (layer "F.Fab")
-      (effects (font (size 1 1) (thickness 0.15)))
-    )
-    (fp_line (start -0.63 -1.27) (end -0.63 1.27) (layer "F.CrtYd") (width 0.05))
-    (fp_line (start 0.63 -1.27) (end -0.63 -1.27) (layer "F.CrtYd") (width 0.05))
-    (fp_line (start 0.63 1.27) (end 0.63 -1.27) (layer "F.CrtYd") (width 0.05))
-    (fp_line (start -0.63 1.27) (end 0.63 1.27) (layer "F.CrtYd") (width 0.05))
-    (fp_line (start 0.63 1.27) (end -0.63 1.27) (layer "F.Fab") (width 0.1))
-    (fp_line (start -0.63 1.27) (end -0.63 -1.27) (layer "F.Fab") (width 0.1))
-    (fp_line (start 0.63 -1.27) (end 0.63 1.27) (layer "F.Fab") (width 0.1))
-    (fp_line (start -0.63 -1.27) (end 0.63 -1.27) (layer "F.Fab") (width 0.1))
-    (pad "1" smd roundrect (at 0 0) (size 1 2) (layers "B.Cu" "B.Mask") (roundrect_rratio 0.25)
-      (net 2 "GND"))
   )
   (footprint "Diode_SMD:D_SOD-123F" (layer "F.Cu")
@@
     )
   )
-  (footprint "motor-mount:motor-mount" (layer "F.Cu")
-    (at 71.2908 73.3298)
-    (property "Sheetfile" "pixel-pump-motor-board.kicad_sch")
-    (property "Sheetname" "")
-    (fp_text reference "J2" (at 8.89 -12.168 unlocked) (layer "F.SilkS") hide
-      (effects (font (size 1 1) (thickness 0.15)))
-    )
-    (fp_text value "motor-connector" (at 8.89 -10.668 unlocked) (layer "F.Fab") hide
-      (effects (font (size 1 1) (thickness 0.15)))
-    )
-    (fp_text user "${REFERENCE}" (at 8.89 -9.168 unlocked) (layer "F.Fab") hide
-      (effects (font (size 1 1) (thickness 0.15)))
-    )
-    (pad "1" thru_hole oval (at 8.77 -5.588) (size 2.8 4.2) (drill oval 1 3) (layers *.Cu "F.Mask") (remove_unused_layers)
-      (net 1 "BEMF_PIN") (pinfunction "motor") (pintype "bidirectional"))
-  )
   (gr_line (start 80.358453 68.668291) (end 80.358453 66.668291) (layer "Dwgs.User") (width 0.2))

Commit message: Minor adjustments and iBOM generation
Parts:
- added J11: Motor Chassis GND, TestPoint:TestPoint_Pad_2.0x2.0mm, B.Cu at (67.5, 58.8)
- added J5: Motor Chassis GND, TestPoint:TestPoint_Pad_2.0x2.0mm, B.Cu at (92.7, 58.7)
- added J7: Motor Chassis GND, TestPoint:TestPoint_Pad_2.0x2.0mm, B.Cu at (80.1, 46.1)
- added J8: Motor Chassis GND, TestPoint:TestPoint_Pad_2.0x2.0mm, B.Cu at (80.0, 71.2)
Routing:
- net GND: vias 23 -> 24
