File: pixel-pump-motor-board.kicad_pcb (KiCad board)
At the start: 2 copper layers, 28.2 x 28.2 mm, 17 parts, among them J1 BM04B-SRSS-TBT(LF)(SN), J11 Motor Chassis GND, J2 motor-connector, J3 motor-connector, J5 Motor Chassis GND, J7 Motor Chassis GND, J8 Motor Chassis GND, Q1 STN4NF20L, U1 250X15W104MV4E

Commit message: Fix bemf pin
Connections:
- C1 pad 1: BEMF_PIN -> +12V
- D1 pad 1: BEMF_PIN -> +12V
- D1 pad 2: Net-(D1-Pad2) -> BEMF_PIN
- J1 pad 1: BEMF_PIN -> +12V
- J2 pad 1: BEMF_PIN -> +12V
- J3 pad 1: Net-(D1-Pad2) -> BEMF_PIN
- Q1 pad 2: Net-(D1-Pad2) -> BEMF_PIN
- Q1 pad T: Net-(D1-Pad2) -> BEMF_PIN
- U1 pad 1: Net-(D1-Pad2) -> BEMF_PIN
- U1 pad 2: BEMF_PIN -> +12V
Routing:
- net Net-(D1-Pad2): track 36.3 -> 0.00 mm, vias 5 -> 0
- net +12V: track 0.00 -> 20.1 mm, vias 0 -> 4
- net BEMF_PIN: track 43.2 -> 46.5 mm

Commit message: Revision bump
Other:
- board text added: "Rev 2"
- board text removed: "Rev 1"
Changed lines of the file:
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@@
     (effects (font (size 0.65 0.65) (thickness 0.13)))
   )
-  (gr_text "Rev 1" (at 69 61.325) (layer "F.SilkS")
+  (gr_text "Rev 2" (at 69 61.325) (layer "F.SilkS")
     (effects (font (size 0.65 0.65) (thickness 0.13)))
   )

Commit message: Remove bemf and add robins logo
Parts:
- removed D2: 2V, Diode_SMD:D_SOD-123
- removed R3: 680k, Resistor_SMD:R_0603_1608Metric
- removed R4: 120k, Resistor_SMD:R_0603_1608Metric
- removed kibuzzard-610914A4: G***, kibuzzard-610914A4
Connections:
- net BEMF_PIN renamed Net-(D1-Pad2)
- J1 pad 3: BEMF -> GND
Routing:
- net BEMF: track 10.3 -> 0.00 mm, vias 2 -> 0
- net Net-(D1-Pad2): track 46.5 -> 36.3 mm, vias 6 -> 5
- net GND: track 1.65 -> 3.23 mm, vias 24 -> 25
Other:
- board text added: "PIXEL PUMP"
- board text added: "REV 3"
- board text removed: "Rev 2"

Commit message: Bump rev
Parts:
- added kibuzzard-62EBC13F: G***, kibuzzard-62EBC13F, F.Cu at (87.0, 50.5)
- added kibuzzard-62EBC161: G***, kibuzzard-62EBC161, F.Cu at (86.3, 52.0)
Other:
- board text removed: "MOTOR DRIVER"
- board text removed: "PIXEL PUMP"

Commit message: Update val to BM04B
Parts:
- J1: value BM04B-SRSS-TBT(LF)(SN) -> BM04B
Changed lines of the file:
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@@
       (effects (font (size 0.65 0.65) (thickness 0.13)))
     )
-    (fp_text value "BM04B-SRSS-TBT(LF)(SN)" (at 0 3.3 90) (layer "F.Fab")
+    (fp_text value "BM04B" (at 0 3.3 90) (layer "F.Fab")
       (effects (font (size 1 1) (thickness 0.15)))
     )

Commit message: Add fiducials, fix SMD/THT, Bump rev to 4
Parts:
- added FID1: Fiducial, Fiducial:Fiducial_0.5mm_Mask1mm, F.Cu at (89.0, 49.7)
- added FID2: Fiducial, Fiducial:Fiducial_0.5mm_Mask1mm, F.Cu at (71.1, 67.6)
Other:
- board text added: "REV 4"
- board text removed: "REV 3"
Changed lines of the file:
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@@
     (property "Sheetfile" "pixel-pump-motor-board.kicad_sch")
     (property "Sheetname" "")
-    (attr through_hole)
+    (attr smd)
     (fp_text reference "U1" (at 2.368808 -0.176777 45) (layer "F.SilkS")
       (effects (font (size 0.65 0.65) (thickness 0.13)))
@@
     (property "Sheetfile" "pixel-pump-motor-board.kicad_sch")
     (property "Sheetname" "")
-    (attr through_hole)
+    (attr smd)
     (fp_text reference "Q1" (at 2.722361 -5.800516 45) (layer "F.SilkS")
       (effects (font (size 0.65 0.65) (thickness 0.13)))
@@
       (net 1 "Net-(D1-Pad2)") (pinfunction "motor") (pintype "bidirectional"))
   )
+  (footprint "Fiducial:Fiducial_0.5mm_Mask1mm" (layer "F.Cu")
+    (at 89.0016 49.6824)
+    (descr "Circular Fiducial, 0.5mm bare copper, 1mm soldermask opening (Level C)")
+    (tags "fiducial")
+    (property "Sheetfile" "pixel-pump-motor-board.kicad_sch")
+    (property "Sheetname" "")
+    (attr smd)
+    (fp_text reference "FID1" (at 0 -1.5) (layer "F.SilkS") hide
+      (effects (font (size 1 1) (thickness 0.15)))
+    )
+    (fp_text value "Fiducial" (at 0 1.5) (layer "F.Fab")
+      (effects (font (size 1 1) (thickness 0.15)))
+    )
+    (fp_text user "${REFERENCE}" (at 0 0) (layer "F.Fab")
+      (effects (font (size 0.2 0.2) (thickness 0.04)))
+    )
+    (fp_circle (center 0 0) (end 0.75 0) (layer "F.CrtYd") (width 0.05) (fill none))
+    (fp_circle (center 0 0) (end 0.5 0) (layer "F.Fab") (width 0.1) (fill none))
+    (pad "" smd circle (at 0 0) (size 0.5 0.5) (layers "F.Cu" "F.Mask")
+      (solder_mask_margin 0.25) (clearance 0.25))
+  )
   (footprint "Capacitor_Tantalum_SMD:CP_EIA-3216-18_Kemet-A" (layer "F.Cu")
     (at 84.3 66.3 135)
@@
     )
   )
+  (footprint "Fiducial:Fiducial_0.5mm_Mask1mm" (layer "F.Cu")
+    (at 71.0792 67.6148)
+    (descr "Circular Fiducial, 0.5mm bare copper, 1mm soldermask opening (Level C)")
+    (tags "fiducial")
+    (property "Sheetfile" "pixel-pump-motor-board.kicad_sch")
+    (property "Sheetname" "")
+    (attr smd)
+    (fp_text reference "FID2" (at 0 -1.5) (layer "F.SilkS") hide
+      (effects (font (size 1 1) (thickness 0.15)))
+    )
+    (fp_text value "Fiducial" (at 0 1.5) (layer "F.Fab")
+      (effects (font (size 1 1) (thickness 0.15)))
+    )
+    (fp_text user "${REFERENCE}" (at 0 0) (layer "F.Fab")
+      (effects (font (size 0.2 0.2) (thickness 0.04)))
+    )
+    (fp_circle (center 0 0) (end 0.75 0) (layer "F.CrtYd") (width 0.05) (fill none))
+    (fp_circle (center 0 0) (end 0.5 0) (layer "F.Fab") (width 0.1) (fill none))
+    (pad "" smd circle (at 0 0) (size 0.5 0.5) (layers "F.Cu" "F.Mask")
+      (solder_mask_margin 0.25) (clearance 0.25))
+  )
   (footprint "motor-mount:motor-mount" (layer "F.Cu")
     (at 71.255 73.263)
@@
   (gr_circle (center 80.108453 58.668291) (end 94.208453 58.668291) (layer "Edge.Cuts") (width 0.2) (fill none))
   (gr_circle (center 80.108453 58.668291) (end 84.358453 58.668291) (layer "Edge.Cuts") (width 0.2) (fill none))
-  (gr_text "REV 3" (at 84.2908 53.2478 -40) (layer "F.SilkS")
+  (gr_text "REV 4" (at 84.2908 53.2478 -40) (layer "F.SilkS")
     (effects (font (size 0.65 0.65) (thickness 0.13)))
   )
@@
     (connect_pads yes (clearance 0))
     (min_thickness 0.254)
-    (keepout (tracks allowed) (vias allowed) (pads allowed ) (copperpour not_allowed) (footprints allowed))
+    (keepout (tracks allowed) (vias allowed) (pads allowed) (copperpour not_allowed) (footprints allowed))
     (fill (thermal_gap 0.508) (thermal_bridge_width 0.508))
     (polygon

Commit message: Add 3rd fiducial
Parts:
- added FID3: Fiducial, Fiducial:Fiducial_0.5mm_Mask1mm, F.Cu at (88.0, 68.5)
Changed lines of the file:
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@@
     )
+  )
+  (footprint "Fiducial:Fiducial_0.5mm_Mask1mm" (layer "F.Cu")
+    (at 87.9856 68.4784)
+    (descr "Circular Fiducial, 0.5mm bare copper, 1mm soldermask opening (Level C)")
+    (tags "fiducial")
+    (property "Sheetfile" "pixel-pump-motor-board.kicad_sch")
+    (property "Sheetname" "")
+    (attr smd)
+    (fp_text reference "FID3" (at 0 -1.5) (layer "F.SilkS") hide
+      (effects (font (size 1 1) (thickness 0.15)))
+    )
+    (fp_text value "Fiducial" (at 0 1.5) (layer "F.Fab")
+      (effects (font (size 1 1) (thickness 0.15)))
+    )
+    (fp_text user "${REFERENCE}" (at 0 0) (layer "F.Fab")
+      (effects (font (size 0.2 0.2) (thickness 0.04)))
+    )
+    (fp_circle (center 0 0) (end 0.75 0) (layer "F.CrtYd") (width 0.05) (fill none))
+    (fp_circle (center 0 0) (end 0.5 0) (layer "F.Fab") (width 0.1) (fill none))
+    (pad "" smd circle (at 0 0) (size 0.5 0.5) (layers "F.Cu" "F.Mask")
+      (solder_mask_margin 0.25) (clearance 0.25))
   )
   (footprint "motor-mount:motor-mount" (layer "F.Cu")

Commit message: Remove unneeded VIA
Routing:
- net GND: track 3.23 -> 1.65 mm, vias 25 -> 24
Other:
- board text added: "REV 5"
- board text removed: "REV 4"
Changed lines of the file:
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@@
     )
     (model "${KIPRJMOD}/components/BM04B-SRSS-TB-LF--SN---3DModel-STEP-56544.STEP"
-      (offset (xyz 0 0 0))
+      (offset (xyz 0 0.5 0))
       (scale (xyz 1 1 1))
       (rotate (xyz -90 0 0))
@@
   (gr_circle (center 80.108453 58.668291) (end 94.208453 58.668291) (layer "Edge.Cuts") (width 0.2) (fill none))
   (gr_circle (center 80.108453 58.668291) (end 84.358453 58.668291) (layer "Edge.Cuts") (width 0.2) (fill none))
-  (gr_text "REV 4" (at 84.2908 53.2478 -40) (layer "F.SilkS")
+  (gr_text "REV 5" (at 84.2908 53.2478 -40) (layer "F.SilkS")
     (effects (font (size 0.65 0.65) (thickness 0.13)))
   )
@@
   (segment (start 74.4 60.925) (end 77.7 64.225) (width 0.5) (layer "B.Cu") (net 1))
   (segment (start 73.35 53.075) (end 76.7934 49.6316) (width 0.5) (layer "B.Cu") (net 1))
-  (segment (start 87.7 58.6) (end 89.275 58.6) (width 0.25) (layer "F.Cu") (net 2))
   (segment (start 85.316283 65.083717) (end 86.483717 63.916283) (width 0.5) (layer "F.Cu") (net 2))
   (via (at 91.422785 52.871178) (size 0.8) (drill 0.4) (layers "F.Cu" "B.Cu") (free) (net 2))
@@
   (via (at 70.19067 66.659475) (size 0.8) (drill 0.4) (layers "F.Cu" "B.Cu") (free) (net 2))
   (via (at 82.073209 71.220754) (size 0.8) (drill 0.4) (layers "F.Cu" "B.Cu") (free) (net 2))
-  (via (at 87.7 58.6) (size 0.8) (drill 0.4) (layers "F.Cu" "B.Cu") (net 2))
   (via (at 72.072182 68.540987) (size 0.8) (drill 0.4) (layers "F.Cu" "B.Cu") (free) (net 2))
   (via (at 68.4276 53.721) (size 0.8) (drill 0.4) (layers "F.Cu" "B.Cu") (free) (net 2))
