File: pixel-pump-motor-board.kicad_pcb (KiCad board)
At the start: 2 copper layers, 28.2 x 28.2 mm, 20 parts, among them J1 BM04B-SRSS-TBT, J11 Motor Chassis GND, J2 motor-connector, J3 motor-connector, J5 Motor Chassis GND, J7 Motor Chassis GND, J8 Motor Chassis GND, Q1 STN4NF20L, T1 Tab, T2 Tab, U1 250X15W104MV4E

Commit message: Add BM04B footprint
Parts:
- moved J1 0.41 mm to (87.5, 59.1)
Changed lines of the file:
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@@
   )
   (footprint "Connector_JST:JST_SH_BM04B-SRSS-TB_1x04-1MP_P1.00mm_Vertical" (layer "F.Cu")
-    (at 87.95 59.1 90)
+    (at 87.5436 59.1 90)
     (descr "JST SH series connector, BM04B-SRSS-TB (http://www.jst-mfg.com/product/pdf/eng/eSH.pdf), generated with kicad-footprint-generator")
     (tags "connector JST SH side entry")
