File: pixel-pump-motor-board.kicad_sch (KiCad schematic)
At the start: 9 parts, among them J2 motor-connector, J3 motor-connector, Q1 STN4NF20L, U1 250X15W104MV4E

Commit message: Finished
Parts:
- removed J?: MOTOR, Connector_JST:JST_SH_BM04B-SRSS-TB_1x04-1MP_P1.00mm_Vertical, symbol Connector_Generic:Conn_01x04
- added J1: BM04B-SRSS-TBT(LF)(SN), Connector_JST:JST_SH_BM04B-SRSS-TB_1x04-1MP_P1.00mm_Vertical, symbol Connector_Generic:Conn_01x04
Connections:
- net +12V: now also J1.1 (Pin_1)
- net BEMF: now also J1.3 (Pin_3)
- net GND: now also J1.4 (Pin_4)
- net PWM: now also J1.2 (Pin_2)
Changed lines of the file:
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@@
     (stroke (width 0) (type solid) (color 0 0 0 0))
   )
-  (wire (pts (xy 47.625 46.99) (xy 58.42 46.99))
-    (stroke (width 0) (type solid) (color 0 0 0 0))
-  )
-  (wire (pts (xy 47.625 49.53) (xy 56.515 49.53))
-    (stroke (width 0) (type solid) (color 0 0 0 0))
-  )
-  (wire (pts (xy 47.625 52.07) (xy 56.515 52.07))
-    (stroke (width 0) (type solid) (color 0 0 0 0))
-  )
-  (wire (pts (xy 47.625 54.61) (xy 58.42 54.61))
-    (stroke (width 0) (type solid) (color 0 0 0 0))
-  )
-  (wire (pts (xy 58.42 46.99) (xy 58.42 43.815))
-    (stroke (width 0) (type solid) (color 0 0 0 0))
-  )
-  (wire (pts (xy 58.42 54.61) (xy 58.42 58.42))
+  (wire (pts (xy 54.61 48.26) (xy 61.595 48.26))
+    (stroke (width 0) (type solid) (color 0 0 0 0))
+  )
+  (wire (pts (xy 54.61 50.8) (xy 61.595 50.8))
+    (stroke (width 0) (type solid) (color 0 0 0 0))
+  )
+  (wire (pts (xy 54.61 53.34) (xy 61.595 53.34))
+    (stroke (width 0) (type solid) (color 0 0 0 0))
+  )
+  (wire (pts (xy 54.61 55.88) (xy 61.595 55.88))
     (stroke (width 0) (type solid) (color 0 0 0 0))
   )
@@
     (stroke (width 0) (type solid) (color 0 0 0 0))
   )
+  (wire (pts (xy 61.595 48.26) (xy 61.595 43.815))
+    (stroke (width 0) (type solid) (color 0 0 0 0))
+  )
+  (wire (pts (xy 61.595 55.88) (xy 61.595 58.42))
+    (stroke (width 0) (type solid) (color 0 0 0 0))
+  )
   (wire (pts (xy 100.33 49.53) (xy 112.395 49.53))
     (stroke (width 0) (type solid) (color 0 0 0 0))
@@
     (stroke (width 0) (type solid) (color 0 0 0 0))
   )
-  (global_label "PWM" (shape input) (at 56.515 49.53 0)
+  (global_label "PWM" (shape input) (at 61.595 50.8 0)
     (effects (font (size 1.27 1.27)) (justify left))
-    (property "Intersheet References" "${INTERSHEET_REFS}" (id 0) (at 282.575 118.11 0)
-      (effects (font (size 1.27 1.27)) hide)
-    )
-  )
-  (global_label "BEMF" (shape input) (at 56.515 52.07 0)
+    (property "Intersheet References" "${INTERSHEET_REFS}" (id 0) (at 287.655 119.38 0)
+      (effects (font (size 1.27 1.27)) hide)
+    )
+  )
+  (global_label "BEMF" (shape input) (at 61.595 53.34 0)
     (effects (font (size 1.27 1.27)) (justify left))
-    (property "Intersheet References" "${INTERSHEET_REFS}" (id 0) (at 282.575 120.65 0)
-      (effects (font (size 1.27 1.27)) hide)
+    (property "Intersheet References" "${INTERSHEET_REFS}" (id 0) (at 73.2731 53.2606 0)
+      (effects (font (size 1.27 1.27)) (justify left) hide)
     )
   )
@@
     (pin "1")
   )
-  (symbol (lib_id "power:+12V") (at 58.42 43.815 0) (unit 1)
-    (in_bom yes) (on_board yes)
-    (property "Reference" "#PWR01" (id 0) (at 58.42 47.625 0)
-      (effects (font (size 1.27 1.27)) hide)
-    )
-    (property "Value" "+12V" (id 1) (at 58.801 39.4208 0))
-    (property "Footprint" "" (id 2) (at 58.42 43.815 0)
-      (effects (font (size 1.27 1.27)) hide)
-    )
-    (property "Datasheet" "" (id 3) (at 58.42 43.815 0)
+  (symbol (lib_id "power:+12V") (at 61.595 43.815 0) (unit 1)
+    (in_bom yes) (on_board yes)
+    (property "Reference" "#PWR0104" (id 0) (at 61.595 47.625 0)
+      (effects (font (size 1.27 1.27)) hide)
+    )
+    (property "Value" "+12V" (id 1) (at 61.976 39.4208 0))
+    (property "Footprint" "" (id 2) (at 61.595 43.815 0)
+      (effects (font (size 1.27 1.27)) hide)
+    )
+    (property "Datasheet" "" (id 3) (at 61.595 43.815 0)
       (effects (font (size 1.27 1.27)) hide)
     )
@@
     (pin "1")
   )
-  (symbol (lib_id "power:GND") (at 58.42 58.42 0) (unit 1)
-    (in_bom yes) (on_board yes)
-    (property "Reference" "#PWR02" (id 0) (at 58.42 64.77 0)
-      (effects (font (size 1.27 1.27)) hide)
-    )
-    (property "Value" "GND" (id 1) (at 58.547 62.8142 0))
-    (property "Footprint" "" (id 2) (at 58.42 58.42 0)
-      (effects (font (size 1.27 1.27)) hide)
-    )
-    (property "Datasheet" "" (id 3) (at 58.42 58.42 0)
-      (effects (font (size 1.27 1.27)) hide)
-    )
-    (pin "1")
-  )
   (symbol (lib_id "power:GND") (at 59.055 85.09 0) (unit 1)
     (in_bom yes) (on_board yes)
@@
     )
     (property "Datasheet" "" (id 3) (at 59.055 85.09 0)
+      (effects (font (size 1.27 1.27)) hide)
+    )
+    (pin "1")
+  )
+  (symbol (lib_id "power:GND") (at 61.595 58.42 0) (unit 1)
+    (in_bom yes) (on_board yes)
+    (property "Reference" "#PWR0103" (id 0) (at 61.595 64.77 0)
+      (effects (font (size 1.27 1.27)) hide)
+    )
+    (property "Value" "GND" (id 1) (at 61.722 62.8142 0))
+    (property "Footprint" "" (id 2) (at 61.595 58.42 0)
+      (effects (font (size 1.27 1.27)) hide)
+    )
+    (property "Datasheet" "" (id 3) (at 61.595 58.42 0)
       (effects (font (size 1.27 1.27)) hide)
     )
@@
     (pin "2")
   )
-  (symbol (lib_id "Connector_Generic:Conn_01x04") (at 42.545 49.53 0) (mirror y) (unit 1)
-    (in_bom yes) (on_board yes)
-    (property "Reference" "J?" (id 0) (at 42.545 59.69 0))
-    (property "Value" "MOTOR" (id 1) (at 40.005 57.785 0))
-    (property "Footprint" "Connector_JST:JST_SH_BM04B-SRSS-TB_1x04-1MP_P1.00mm_Vertical" (id 2) (at 42.545 49.53 0)
-      (effects (font (size 1.27 1.27)) hide)
-    )
-    (property "Datasheet" "~" (id 3) (at 42.545 49.53 0)
-      (effects (font (size 1.27 1.27)) hide)
-    )
-    (property "Source" "https://lcsc.com/product-detail/Wire-To-Board-Wire-To-Wire-Connector_BOOMELE-Boom-Precision-Elec-C145961_C145961.html" (id 4) (at 42.545 49.53 0)
+  (symbol (lib_id "Connector_Generic:Conn_01x04") (at 49.53 50.8 0) (mirror y) (unit 1)
+    (in_bom yes) (on_board yes)
+    (property "Reference" "J1" (id 0) (at 49.53 60.96 0))
+    (property "Value" "BM04B-SRSS-TBT(LF)(SN)" (id 1) (at 38.735 59.055 0))
+    (property "Footprint" "Connector_JST:JST_SH_BM04B-SRSS-TB_1x04-1MP_P1.00mm_Vertical" (id 2) (at 49.53 50.8 0)
+      (effects (font (size 1.27 1.27)) hide)
+    )
+    (property "Datasheet" "~" (id 3) (at 49.53 50.8 0)
+      (effects (font (size 1.27 1.27)) hide)
+    )
+    (property "Source" "https://lcsc.com/product-detail/Wire-To-Board-Wire-To-Wire-Connector_BOOMELE-Boom-Precision-Elec-C145961_C145961.html" (id 4) (at 49.53 50.8 0)
       (effects (font (size 1.27 1.27)) hide)
     )
@@
       (reference "#FLG0102") (unit 1) (value "PWR_FLAG") (footprint "")
     )
-    (path "/7c1f7596-2adc-4ddd-81b2-8364f9dd10e7"
-      (reference "#PWR01") (unit 1) (value "+12V") (footprint "")
-    )
-    (path "/fe4571d6-4bac-4c5e-995d-3b824025cf76"
-      (reference "#PWR02") (unit 1) (value "GND") (footprint "")
-    )
     (path "/0bd113ac-c401-4364-b116-e3829096fe8c"
       (reference "#PWR03") (unit 1) (value "+12V") (footprint "")
@@
       (reference "#PWR0102") (unit 1) (value "GND") (footprint "")
     )
+    (path "/0777afb6-c9f5-40d3-a69c-cf76b40a7a2d"
+      (reference "#PWR0103") (unit 1) (value "GND") (footprint "")
+    )
+    (path "/bd142016-c6ea-444a-843a-17a19fa62852"
+      (reference "#PWR0104") (unit 1) (value "+12V") (footprint "")
+    )
     (path "/1f7a19e5-e285-4bb1-bf4e-7d1ea9a40a35"
       (reference "C1") (unit 1) (value "C_Polarized") (footprint "Capacitor_Tantalum_SMD:CP_EIA-3216-18_Kemet-A")
@@
       (reference "D1") (unit 1) (value "SOD4007") (footprint "Diode_SMD:D_SOD-123F")
     )
+    (path "/80f92d9a-5f30-4aa7-abbe-2a03b44d3c62"
+      (reference "J1") (unit 1) (value "BM04B-SRSS-TBT(LF)(SN)") (footprint "Connector_JST:JST_SH_BM04B-SRSS-TB_1x04-1MP_P1.00mm_Vertical")
+    )
     (path "/d44ad972-8a51-43a4-b571-d28629d63fde"
       (reference "J2") (unit 1) (value "motor-connector") (footprint "motor-mount:motor-mount")
@@
       (reference "J3") (unit 1) (value "motor-connector") (footprint "motor-mount:motor-mount")
     )
-    (path "/d396a52b-e83f-4e49-aa4f-d1d81b7134a9"
-      (reference "J?") (unit 1) (value "MOTOR") (footprint "Connector_JST:JST_SH_BM04B-SRSS-TB_1x04-1MP_P1.00mm_Vertical")
-    )
     (path "/027211cc-9745-45fd-aa4e-2bf54759e7b3"

Commit message: Finish motor board
Parts:
- added D2: 2V, Diode_SMD:D_SOD-123, symbol Device:D_Zener
- added R3: 680k, Resistor_SMD:R_0603_1608Metric, symbol Device:R
- added R4: 120k, Resistor_SMD:R_0603_1608Metric, symbol Device:R
Connections:
- net +12V: now also R3.1
- net BEMF: now also D2.1 (K), R3.2, R4.1
- net GND: now also D2.2 (A), R4.2
Other:
- note added: "Back EMF voltage divider"
- note added: "Vadc = Vmotor * ( 120k / ( 680k + 120k ) )"
- note added: "Vmotor = 12V Vadc = 1.8V"
Changed lines of the file:
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@@
 (kicad_sch (version 20210621) (generator eeschema)
   (paper "A4")
+  (junction (at 57.785 150.495) (diameter 0.9144) (color 0 0 0 0))
+  (junction (at 57.785 163.195) (diameter 0.9144) (color 0 0 0 0))
+  (junction (at 69.85 150.495) (diameter 0.9144) (color 0 0 0 0))
+  (junction (at 103.505 49.53) (diameter 0.9144) (color 0 0 0 0))
   (junction (at 112.395 49.53) (diameter 0.9144) (color 0 0 0 0))
   (junction (at 112.395 59.69) (diameter 0.9144) (color 0 0 0 0))
@@
     (stroke (width 0) (type solid) (color 0 0 0 0))
   )
+  (wire (pts (xy 57.785 136.525) (xy 57.785 140.335))
+    (stroke (width 0) (type solid) (color 0 0 0 0))
+  )
+  (wire (pts (xy 57.785 147.955) (xy 57.785 150.495))
+    (stroke (width 0) (type solid) (color 0 0 0 0))
+  )
+  (wire (pts (xy 57.785 150.495) (xy 57.785 153.67))
+    (stroke (width 0) (type solid) (color 0 0 0 0))
+  )
+  (wire (pts (xy 57.785 150.495) (xy 69.85 150.495))
+    (stroke (width 0) (type solid) (color 0 0 0 0))
+  )
+  (wire (pts (xy 57.785 161.29) (xy 57.785 163.195))
+    (stroke (width 0) (type solid) (color 0 0 0 0))
+  )
+  (wire (pts (xy 57.785 163.195) (xy 57.785 164.465))
+    (stroke (width 0) (type solid) (color 0 0 0 0))
+  )
+  (wire (pts (xy 57.785 163.195) (xy 69.85 163.195))
+    (stroke (width 0) (type solid) (color 0 0 0 0))
+  )
   (wire (pts (xy 59.055 78.74) (xy 59.055 85.09))
     (stroke (width 0) (type solid) (color 0 0 0 0))
@@
     (stroke (width 0) (type solid) (color 0 0 0 0))
   )
-  (wire (pts (xy 100.33 49.53) (xy 112.395 49.53))
+  (wire (pts (xy 69.85 150.495) (xy 69.85 153.67))
+    (stroke (width 0) (type solid) (color 0 0 0 0))
+  )
+  (wire (pts (xy 69.85 150.495) (xy 76.2 150.495))
+    (stroke (width 0) (type solid) (color 0 0 0 0))
+  )
+  (wire (pts (xy 69.85 161.29) (xy 69.85 163.195))
+    (stroke (width 0) (type solid) (color 0 0 0 0))
+  )
+  (wire (pts (xy 100.33 49.53) (xy 103.505 49.53))
     (stroke (width 0) (type solid) (color 0 0 0 0))
   )
@@
     (stroke (width 0) (type solid) (color 0 0 0 0))
   )
+  (wire (pts (xy 103.505 45.72) (xy 103.505 49.53))
+    (stroke (width 0) (type solid) (color 0 0 0 0))
+  )
+  (wire (pts (xy 103.505 49.53) (xy 112.395 49.53))
+    (stroke (width 0) (type solid) (color 0 0 0 0))
+  )
   (wire (pts (xy 105.41 54.61) (xy 107.315 54.61))
     (stroke (width 0) (type solid) (color 0 0 0 0))
@@
   (wire (pts (xy 158.115 63.5) (xy 158.115 59.69))
     (stroke (width 0) (type solid) (color 0 0 0 0))
+  )
+  (polyline (pts (xy 12.065 100.965) (xy 95.25 100.965))
+    (stroke (width 0) (type dash) (color 0 0 0 0))
+  )
+  (polyline (pts (xy 95.25 100.965) (xy 95.25 197.485))
+    (stroke (width 0) (type dash) (color 0 0 0 0))
+  )
+  (text "Back EMF voltage divider" (at 14.605 107.315 0)
+    (effects (font (size 2 2)) (justify left bottom))
+  )
+  (text "Vmotor = 12V\nVadc = 1.8V" (at 22.225 180.975 0)
+    (effects (font (size 1.27 1.27)) (justify left bottom))
+  )
+  (text "Vadc = Vmotor * ( 120k / ( 680k + 120k ) )" (at 22.225 184.785 0)
+    (effects (font (size 1.27 1.27)) (justify left bottom))
+  )
+  (global_label "BEMF_PIN" (shape input) (at 57.785 136.525 90) (fields_autoplaced)
+    (effects (font (size 1.27 1.27)) (justify left))
+    (property "Intersheet References" "${INTERSHEET_REFS}" (id 0) (at 57.7056 124.98 90)
+      (effects (font (size 1.27 1.27)) (justify left) hide)
+    )
   )
   (global_label "PWM" (shape input) (at 61.595 50.8 0)
@@
     )
   )
+  (global_label "BEMF" (shape input) (at 76.2 150.495 0)
+    (effects (font (size 1.27 1.27)) (justify left))
+    (property "Intersheet References" "${INTERSHEET_REFS}" (id 0) (at 87.8781 150.4156 0)
+      (effects (font (size 1.27 1.27)) (justify left) hide)
+    )
+  )
+  (global_label "BEMF_PIN" (shape input) (at 103.505 45.72 90) (fields_autoplaced)
+    (effects (font (size 1.27 1.27)) (justify left))
+    (property "Intersheet References" "${INTERSHEET_REFS}" (id 0) (at 103.4256 34.175 90)
+      (effects (font (size 1.27 1.27)) (justify left) hide)
+    )
+  )
   (global_label "PWM" (shape input) (at 126.365 88.9 270)
     (effects (font (size 1.27 1.27)) (justify right))
@@
     (pin "1")
   )
+  (symbol (lib_id "power:GND") (at 57.785 164.465 0) (unit 1)
+    (in_bom yes) (on_board yes)
+    (property "Reference" "#PWR01" (id 0) (at 57.785 170.815 0)
+      (effects (font (size 1.27 1.27)) hide)
+    )
+    (property "Value" "GND" (id 1) (at 57.912 168.8592 0))
+    (property "Footprint" "" (id 2) (at 57.785 164.465 0)
+      (effects (font (size 1.27 1.27)) hide)
+    )
+    (property "Datasheet" "" (id 3) (at 57.785 164.465 0)
+      (effects (font (size 1.27 1.27)) hide)
+    )
+    (pin "1")
+  )
   (symbol (lib_id "power:GND") (at 59.055 85.09 0) (unit 1)
     (in_bom yes) (on_board yes)
@@
     (pin "1")
   )
+  (symbol (lib_id "Device:R") (at 57.785 144.145 0) (unit 1)
+    (in_bom yes) (on_board yes) (fields_autoplaced)
+    (property "Reference" "R3" (id 0) (at 60.325 142.8749 0)
+      (effects (font (size 1.27 1.27)) (justify left))
+    )
+    (property "Value" "680k" (id 1) (at 60.325 145.4149 0)
+      (effects (font (size 1.27 1.27)) (justify left))
+    )
+    (property "Footprint" "Resistor_SMD:R_0603_1608Metric" (id 2) (at 56.007 144.145 90)
+      (effects (font (size 1.27 1.27)) hide)
+    )
+    (property "Datasheet" "~" (id 3) (at 57.785 144.145 0)
+      (effects (font (size 1.27 1.27)) hide)
+    )
+    (pin "1")
+    (pin "2")
+  )
+  (symbol (lib_id "Device:R") (at 57.785 157.48 0) (unit 1)
+    (in_bom yes) (on_board yes) (fields_autoplaced)
+    (property "Reference" "R4" (id 0) (at 60.325 156.2099 0)
+      (effects (font (size 1.27 1.27)) (justify left))
+    )
+    (property "Value" "120k" (id 1) (at 60.325 158.7499 0)
+      (effects (font (size 1.27 1.27)) (justify left))
+    )
+    (property "Footprint" "Resistor_SMD:R_0603_1608Metric" (id 2) (at 56.007 157.48 90)
+      (effects (font (size 1.27 1.27)) hide)
+    )
+    (property "Datasheet" "~" (id 3) (at 57.785 157.48 0)
+      (effects (font (size 1.27 1.27)) hide)
+    )
+    (pin "1")
+    (pin "2")
+  )
   (symbol (lib_id "Device:R") (at 126.365 82.55 0) (unit 1)
     (in_bom yes) (on_board yes)
@@
     )
     (property "Datasheet" "~" (id 3) (at 133.985 81.28 0)
+      (effects (font (size 1.27 1.27)) hide)
+    )
+    (pin "1")
+    (pin "2")
+  )
+  (symbol (lib_id "Device:D_Zener") (at 69.85 157.48 270) (unit 1)
+    (in_bom yes) (on_board yes) (fields_autoplaced)
+    (property "Reference" "D2" (id 0) (at 73.025 156.2099 90)
+      (effects (font (size 1.27 1.27)) (justify left))
+    )
+    (property "Value" "2V" (id 1) (at 73.025 158.7499 90)
+      (effects (font (size 1.27 1.27)) (justify left))
+    )
+    (property "Footprint" "Diode_SMD:D_SOD-123" (id 2) (at 69.85 157.48 0)
+      (effects (font (size 1.27 1.27)) hide)
+    )
+    (property "Datasheet" "~" (id 3) (at 69.85 157.48 0)
       (effects (font (size 1.27 1.27)) hide)
     )
@@
       (reference "#FLG0102") (unit 1) (value "PWR_FLAG") (footprint "")
     )
+    (path "/c4999f21-9844-497b-94a0-2c4bed12bb2d"
+      (reference "#PWR01") (unit 1) (value "GND") (footprint "")
+    )
     (path "/0bd113ac-c401-4364-b116-e3829096fe8c"
       (reference "#PWR03") (unit 1) (value "+12V") (footprint "")
@@
       (reference "D1") (unit 1) (value "SOD4007") (footprint "Diode_SMD:D_SOD-123F")
     )
+    (path "/2b33ce0e-5667-4cbc-a468-321807731f84"
+      (reference "D2") (unit 1) (value "2V") (footprint "Diode_SMD:D_SOD-123")
+    )
     (path "/80f92d9a-5f30-4aa7-abbe-2a03b44d3c62"
       (reference "J1") (unit 1) (value "BM04B-SRSS-TBT(LF)(SN)") (footprint "Connector_JST:JST_SH_BM04B-SRSS-TB_1x04-1MP_P1.00mm_Vertical")
@@
       (reference "R2") (unit 1) (value "100k") (footprint "Resistor_SMD:R_0603_1608Metric")
     )
+    (path "/67192752-d1b9-4bd9-ac5c-b7c9c3082ac3"
+      (reference "R3") (unit 1) (value "680k") (footprint "Resistor_SMD:R_0603_1608Metric")
+    )
+    (path "/2dfd6a67-0fb9-4906-9024-38dde8fc0a5d"
+      (reference "R4") (unit 1) (value "120k") (footprint "Resistor_SMD:R_0603_1608Metric")
+    )
     (path "/c99d9ee8-b4c6-4374-bb5b-0809ce253ad3"

Commit message: Cleanup and generate iBOM
Parts:
- C1: value C_Polarized -> 100n 25V
Changed lines of the file:
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@@
   (symbol (lib_id "motor-mount:motor-connector") (at 99.06 49.53 180) (unit 1)
     (in_bom yes) (on_board yes)
-    (property "Reference" "J2" (id 0) (at 95.885 45.72 0))
-    (property "Value" "motor-connector" (id 1) (at 89.535 47.625 0))
+    (property "Reference" "J2" (id 0) (at 99.06 44.45 0))
+    (property "Value" "motor-connector" (id 1) (at 92.075 46.99 0))
     (property "Footprint" "motor-mount:motor-mount" (id 2) (at 99.06 49.53 0)
       (effects (font (size 1.27 1.27)) hide)
@@
   (symbol (lib_id "motor-mount:motor-connector") (at 99.06 59.69 180) (unit 1)
     (in_bom yes) (on_board yes)
-    (property "Reference" "J3" (id 0) (at 95.885 63.5 0))
-    (property "Value" "motor-connector" (id 1) (at 89.535 61.595 0))
+    (property "Reference" "J3" (id 0) (at 99.06 54.61 0))
+    (property "Value" "motor-connector" (id 1) (at 92.075 57.15 0))
     (property "Footprint" "motor-mount:motor-mount" (id 2) (at 99.06 59.69 0)
       (effects (font (size 1.27 1.27)) hide)
@@
       (effects (font (size 1.27 1.27)) (justify left))
     )
-    (property "Value" "C_Polarized" (id 1) (at 161.925 57.7849 0)
+    (property "Value" "100n 25V" (id 1) (at 161.925 57.7849 0)
       (effects (font (size 1.27 1.27)) (justify left))
     )
@@
     )
     (path "/1f7a19e5-e285-4bb1-bf4e-7d1ea9a40a35"
-      (reference "C1") (unit 1) (value "C_Polarized") (footprint "Capacitor_Tantalum_SMD:CP_EIA-3216-18_Kemet-A")
+      (reference "C1") (unit 1) (value "100n 25V") (footprint "Capacitor_Tantalum_SMD:CP_EIA-3216-18_Kemet-A")
     )
     (path "/0e0e6608-be18-4a36-8a5f-fc659e496bef"
@@
       (reference "J1") (unit 1) (value "BM04B-SRSS-TBT(LF)(SN)") (footprint "Connector_JST:JST_SH_BM04B-SRSS-TB_1x04-1MP_P1.00mm_Vertical")
     )
-    (path "/d44ad972-8a51-43a4-b571-d28629d63fde"
+    (path "/487963d3-ed36-4ffe-bbc0-8af87b349b27"
       (reference "J2") (unit 1) (value "motor-connector") (footprint "motor-mount:motor-mount")
     )
-    (path "/047b9ede-dc55-4807-a86d-647ff742c18f"
+    (path "/c332f8cc-90f7-4adf-b7c8-5b9cae9f618d"
       (reference "J3") (unit 1) (value "motor-connector") (footprint "motor-mount:motor-mount")
     )
