File: pixel-pump-motor-board.kicad_sch (KiCad schematic)
At the start: 12 parts, among them J1 BM04B-SRSS-TBT(LF)(SN), J2 motor-connector, J3 motor-connector, Q1 STN4NF20L, U1 250X15W104MV4E

Commit message: Minor adjustments and iBOM generation
Parts:
- added J11, J5, J7, J8: Motor Chassis GND, TestPoint:TestPoint_Pad_2.0x2.0mm, symbol Connector:Conn_01x01_Male
- J2, J3: now left out of the parts list
Connections:
- net GND: now also J11.1 (Pin_1), J5.1 (Pin_1), J7.1 (Pin_1), J8.1 (Pin_1)
Changed lines of the file:
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@@
+    (stroke (width 0) (type solid) (color 0 0 0 0))
+  )
+  (wire (pts (xy 118.11 130.81) (xy 118.11 137.16))
     (stroke (width 0) (type solid) (color 0 0 0 0))
   )
@@
     (stroke (width 0) (type solid) (color 0 0 0 0))
   )
+  (wire (pts (xy 137.795 130.81) (xy 137.795 137.16))
+    (stroke (width 0) (type solid) (color 0 0 0 0))
+  )
   (wire (pts (xy 142.875 49.53) (xy 142.875 46.99))
     (stroke (width 0) (type solid) (color 0 0 0 0))
@@
     (stroke (width 0) (type solid) (color 0 0 0 0))
   )
+  (wire (pts (xy 156.845 130.81) (xy 156.845 137.16))
+    (stroke (width 0) (type solid) (color 0 0 0 0))
+  )
   (wire (pts (xy 158.115 49.53) (xy 142.875 49.53))
     (stroke (width 0) (type solid) (color 0 0 0 0))
@@
   )
   (wire (pts (xy 158.115 63.5) (xy 158.115 59.69))
+    (stroke (width 0) (type solid) (color 0 0 0 0))
+  )
+  (wire (pts (xy 176.53 130.81) (xy 176.53 137.16))
     (stroke (width 0) (type solid) (color 0 0 0 0))
   )
@@
   )
   (symbol (lib_id "motor-mount:motor-connector") (at 99.06 49.53 180) (unit 1)
-    (in_bom yes) (on_board yes)
+    (in_bom no) (on_board yes)
     (property "Reference" "J2" (id 0) (at 99.06 44.45 0))
     (property "Value" "motor-connector" (id 1) (at 92.075 46.99 0))
@@
   )
   (symbol (lib_id "motor-mount:motor-connector") (at 99.06 59.69 180) (unit 1)
-    (in_bom yes) (on_board yes)
+    (in_bom no) (on_board yes)
     (property "Reference" "J3" (id 0) (at 99.06 54.61 0))
     (property "Value" "motor-connector" (id 1) (at 92.075 57.15 0))
@@
     (pin "1")
   )
+  (symbol (lib_id "Connector:Conn_01x01_Male") (at 118.11 125.73 270) (unit 1)
+    (in_bom yes) (on_board yes)
+    (property "Reference" "J5" (id 0) (at 116.84 124.6123 90)
+      (effects (font (size 1.27 1.27)) (justify left))
+    )
+    (property "Value" "Motor Chassis GND" (id 1) (at 109.22 122.7073 90)
+      (effects (font (size 1.27 1.27)) (justify left))
+    )
+    (property "Footprint" "TestPoint:TestPoint_Pad_2.0x2.0mm" (id 2) (at 118.11 125.73 0)
+      (effects (font (size 1.27 1.27)) hide)
+    )
+    (property "Datasheet" "~" (id 3) (at 118.11 125.73 0)
+      (effects (font (size 1.27 1.27)) hide)
+    )
+    (pin "1")
+  )
+  (symbol (lib_id "Connector:Conn_01x01_Male") (at 137.795 125.73 270) (unit 1)
+    (in_bom yes) (on_board yes)
+    (property "Reference" "J7" (id 0) (at 136.525 124.6123 90)
+      (effects (font (size 1.27 1.27)) (justify left))
+    )
+    (property "Value" "Motor Chassis GND" (id 1) (at 128.905 122.7073 90)
+      (effects (font (size 1.27 1.27)) (justify left))
+    )
+    (property "Footprint" "TestPoint:TestPoint_Pad_2.0x2.0mm" (id 2) (at 137.795 125.73 0)
+      (effects (font (size 1.27 1.27)) hide)
+    )
+    (property "Datasheet" "~" (id 3) (at 137.795 125.73 0)
+      (effects (font (size 1.27 1.27)) hide)
+    )
+    (pin "1")
+  )
+  (symbol (lib_id "Connector:Conn_01x01_Male") (at 156.845 125.73 270) (unit 1)
+    (in_bom yes) (on_board yes)
+    (property "Reference" "J8" (id 0) (at 155.575 124.6123 90)
+      (effects (font (size 1.27 1.27)) (justify left))
+    )
+    (property "Value" "Motor Chassis GND" (id 1) (at 147.955 122.7073 90)
+      (effects (font (size 1.27 1.27)) (justify left))
+    )
+    (property "Footprint" "TestPoint:TestPoint_Pad_2.0x2.0mm" (id 2) (at 156.845 125.73 0)
+      (effects (font (size 1.27 1.27)) hide)
+    )
+    (property "Datasheet" "~" (id 3) (at 156.845 125.73 0)
+      (effects (font (size 1.27 1.27)) hide)
+    )
+    (pin "1")
+  )
+  (symbol (lib_id "Connector:Conn_01x01_Male") (at 176.53 125.73 270) (unit 1)
+    (in_bom yes) (on_board yes)
+    (property "Reference" "J11" (id 0) (at 175.26 124.6123 90)
+      (effects (font (size 1.27 1.27)) (justify left))
+    )
+    (property "Value" "Motor Chassis GND" (id 1) (at 167.64 122.7073 90)
+      (effects (font (size 1.27 1.27)) (justify left))
+    )
+    (property "Footprint" "TestPoint:TestPoint_Pad_2.0x2.0mm" (id 2) (at 176.53 125.73 0)
+      (effects (font (size 1.27 1.27)) hide)
+    )
+    (property "Datasheet" "~" (id 3) (at 176.53 125.73 0)
+      (effects (font (size 1.27 1.27)) hide)
+    )
+    (pin "1")
+  )
   (symbol (lib_id "power:+12V") (at 46.99 84.455 180) (unit 1)
     (in_bom yes) (on_board yes)
@@
     (pin "1")
   )
+  (symbol (lib_id "power:GND") (at 118.11 137.16 0) (unit 1)
+    (in_bom yes) (on_board yes)
+    (property "Reference" "#PWR0105" (id 0) (at 118.11 143.51 0)
+      (effects (font (size 1.27 1.27)) hide)
+    )
+    (property "Value" "GND" (id 1) (at 118.237 141.5542 0))
+    (property "Footprint" "" (id 2) (at 118.11 137.16 0)
+      (effects (font (size 1.27 1.27)) hide)
+    )
+    (property "Datasheet" "" (id 3) (at 118.11 137.16 0)
+      (effects (font (size 1.27 1.27)) hide)
+    )
+    (pin "1")
+  )
   (symbol (lib_id "power:GND") (at 120.015 62.865 0) (unit 1)
     (in_bom yes) (on_board yes)
@@
     (pin "1")
   )
+  (symbol (lib_id "power:GND") (at 137.795 137.16 0) (unit 1)
+    (in_bom yes) (on_board yes)
+    (property "Reference" "#PWR0108" (id 0) (at 137.795 143.51 0)
+      (effects (font (size 1.27 1.27)) hide)
+    )
+    (property "Value" "GND" (id 1) (at 137.922 141.5542 0))
+    (property "Footprint" "" (id 2) (at 137.795 137.16 0)
+      (effects (font (size 1.27 1.27)) hide)
+    )
+    (property "Datasheet" "" (id 3) (at 137.795 137.16 0)
+      (effects (font (size 1.27 1.27)) hide)
+    )
+    (pin "1")
+  )
   (symbol (lib_id "power:GND") (at 142.875 86.36 0) (unit 1)
     (in_bom yes) (on_board yes)
@@
     (pin "1")
   )
+  (symbol (lib_id "power:GND") (at 156.845 137.16 0) (unit 1)
+    (in_bom yes) (on_board yes)
+    (property "Reference" "#PWR0109" (id 0) (at 156.845 143.51 0)
+      (effects (font (size 1.27 1.27)) hide)
+    )
+    (property "Value" "GND" (id 1) (at 156.972 141.5542 0))
+    (property "Footprint" "" (id 2) (at 156.845 137.16 0)
+      (effects (font (size 1.27 1.27)) hide)
+    )
+    (property "Datasheet" "" (id 3) (at 156.845 137.16 0)
+      (effects (font (size 1.27 1.27)) hide)
+    )
+    (pin "1")
+  )
   (symbol (lib_id "power:GND") (at 158.115 63.5 0) (unit 1)
     (in_bom yes) (on_board yes)
@@
     )
     (property "Datasheet" "" (id 3) (at 158.115 63.5 0)
+      (effects (font (size 1.27 1.27)) hide)
+    )
+    (pin "1")
+  )
+  (symbol (lib_id "power:GND") (at 176.53 137.16 0) (unit 1)
+    (in_bom yes) (on_board yes)
+    (property "Reference" "#PWR0112" (id 0) (at 176.53 143.51 0)
+      (effects (font (size 1.27 1.27)) hide)
+    )
+    (property "Value" "GND" (id 1) (at 176.657 141.5542 0))
+    (property "Footprint" "" (id 2) (at 176.53 137.16 0)
+      (effects (font (size 1.27 1.27)) hide)
+    )
+    (property "Datasheet" "" (id 3) (at 176.53 137.16 0)
       (effects (font (size 1.27 1.27)) hide)
     )
@@
       (reference "#PWR0104") (unit 1) (value "+12V") (footprint "")
     )
+    (path "/a7e5c194-fc12-4e92-84da-44e59bbf0abd"
+      (reference "#PWR0105") (unit 1) (value "GND") (footprint "")
+    )
+    (path "/70189bb7-625e-4094-b765-15a0b32e11ab"
+      (reference "#PWR0108") (unit 1) (value "GND") (footprint "")
+    )
+    (path "/72ce30fb-cb15-4d74-917f-74da144616b1"
+      (reference "#PWR0109") (unit 1) (value "GND") (footprint "")
+    )
+    (path "/f0f9aa13-a43a-4673-a341-920fc56f6f40"
+      (reference "#PWR0112") (unit 1) (value "GND") (footprint "")
+    )
     (path "/1f7a19e5-e285-4bb1-bf4e-7d1ea9a40a35"
       (reference "C1") (unit 1) (value "100n 25V") (footprint "Capacitor_Tantalum_SMD:CP_EIA-3216-18_Kemet-A")
@@
       (reference "J3") (unit 1) (value "motor-connector") (footprint "motor-mount:motor-mount")
     )
+    (path "/0f85a9e8-a131-4f43-91b9-1eb38bc085ab"
+      (reference "J5") (unit 1) (value "Motor Chassis GND") (footprint "TestPoint:TestPoint_Pad_2.0x2.0mm")
+    )
+    (path "/09fda414-9fa7-4039-9964-173d7558ba48"
+      (reference "J7") (unit 1) (value "Motor Chassis GND") (footprint "TestPoint:TestPoint_Pad_2.0x2.0mm")
+    )
+    (path "/9dd977ef-21d9-4da8-a2b7-95e48368de34"
+      (reference "J8") (unit 1) (value "Motor Chassis GND") (footprint "TestPoint:TestPoint_Pad_2.0x2.0mm")
+    )
+    (path "/9fc21aca-0720-4bc9-acc9-d4f522fbd7bc"
+      (reference "J11") (unit 1) (value "Motor Chassis GND") (footprint "TestPoint:TestPoint_Pad_2.0x2.0mm")
+    )
     (path "/027211cc-9745-45fd-aa4e-2bf54759e7b3"
