File: pixel-pump-motor-board.kicad_sch (KiCad schematic)
At the start: 16 parts, among them J1 BM04B-SRSS-TBT(LF)(SN), J11 Motor Chassis GND, J2 motor-connector, J3 motor-connector, J5 Motor Chassis GND, J7 Motor Chassis GND, J8 Motor Chassis GND, Q1 STN4NF20L, U1 250X15W104MV4E

Commit message: Fix bemf pin
Connections:
- net +12V: no longer R3.1
- net BEMF_PIN: now reaches D1.2 (A), J3.1 (motor), Q1.2, Q1.T, U1.1
- net BEMF_PIN: now also R3.1
Other:
- moved on the sheet: J2, J3
Changed lines of the file:
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@@
   (junction (at 142.875 59.69) (diameter 0.9144) (color 0 0 0 0)
   )
+  (junction (at 99.06 59.69) (diameter 0) (color 0 0 0 0)
+  )
   (junction (at 69.85 150.495) (diameter 0.9144) (color 0 0 0 0)
   )
-  (junction (at 103.505 49.53) (diameter 0.9144) (color 0 0 0 0)
-  )
-  (wire (pts (xy 100.33 59.69) (xy 112.395 59.69))
+  (wire (pts (xy 96.52 59.69) (xy 99.06 59.69))
     (stroke (width 0) (type solid) (color 0 0 0 0))
   )
@@
     (stroke (width 0) (type solid) (color 0 0 0 0))
   )
+  (wire (pts (xy 99.06 59.69) (xy 112.395 59.69))
+    (stroke (width 0) (type solid) (color 0 0 0 0))
+  )
   (wire (pts (xy 61.595 55.88) (xy 61.595 58.42))
     (stroke (width 0) (type solid) (color 0 0 0 0))
@@
     (stroke (width 0) (type solid) (color 0 0 0 0))
   )
-  (wire (pts (xy 100.33 49.53) (xy 103.505 49.53))
-    (stroke (width 0) (type solid) (color 0 0 0 0))
-  )
-  (wire (pts (xy 103.505 49.53) (xy 112.395 49.53))
+  (wire (pts (xy 96.52 49.53) (xy 112.395 49.53))
     (stroke (width 0) (type solid) (color 0 0 0 0))
   )
@@
     (stroke (width 0) (type solid) (color 0 0 0 0))
   )
-  (wire (pts (xy 103.505 45.72) (xy 103.505 49.53))
-    (stroke (width 0) (type solid) (color 0 0 0 0))
-  )
   (wire (pts (xy 54.61 53.34) (xy 61.595 53.34))
     (stroke (width 0) (type solid) (color 0 0 0 0))
@@
   (wire (pts (xy 142.875 49.53) (xy 142.875 46.99))
     (stroke (width 0) (type solid) (color 0 0 0 0))
+  )
+  (wire (pts (xy 99.06 59.69) (xy 99.06 65.405))
+    (stroke (width 0) (type default) (color 0 0 0 0))
   )
   (wire (pts (xy 133.985 85.09) (xy 133.985 85.725))
@@
     )
   )
-  (global_label "BEMF_PIN" (shape input) (at 103.505 45.72 90) (fields_autoplaced)
-    (effects (font (size 1.27 1.27)) (justify left))
-    (property "Intersheet References" "${INTERSHEET_REFS}" (id 0) (at 103.4256 34.175 90)
-      (effects (font (size 1.27 1.27)) (justify left) hide)
+  (global_label "BEMF_PIN" (shape input) (at 99.06 65.405 270) (fields_autoplaced)
+    (effects (font (size 1.27 1.27)) (justify right))
+    (property "Intersheet References" "${INTERSHEET_REFS}" (id 0) (at 99.1394 76.95 90)
+      (effects (font (size 1.27 1.27)) (justify right) hide)
     )
   )
@@
     (pin "1")
   )
-  (symbol (lib_id "motor-mount:motor-connector") (at 99.06 49.53 180) (unit 1)
+  (symbol (lib_id "motor-mount:motor-connector") (at 95.25 49.53 180) (unit 1)
     (in_bom no) (on_board yes)
-    (property "Reference" "J2" (id 0) (at 99.06 44.45 0))
-    (property "Value" "motor-connector" (id 1) (at 92.075 46.99 0))
-    (property "Footprint" "motor-mount:motor-mount" (id 2) (at 99.06 49.53 0)
-      (effects (font (size 1.27 1.27)) hide)
-    )
-    (property "Datasheet" "" (id 3) (at 99.06 49.53 0)
+    (property "Reference" "J2" (id 0) (at 95.25 44.45 0))
+    (property "Value" "motor-connector" (id 1) (at 88.265 46.99 0))
+    (property "Footprint" "motor-mount:motor-mount" (id 2) (at 95.25 49.53 0)
+      (effects (font (size 1.27 1.27)) hide)
+    )
+    (property "Datasheet" "" (id 3) (at 95.25 49.53 0)
       (effects (font (size 1.27 1.27)) hide)
     )
@@
     (pin "1")
   )
-  (symbol (lib_id "motor-mount:motor-connector") (at 99.06 59.69 180) (unit 1)
+  (symbol (lib_id "motor-mount:motor-connector") (at 95.25 59.69 180) (unit 1)
     (in_bom no) (on_board yes)
-    (property "Reference" "J3" (id 0) (at 99.06 54.61 0))
-    (property "Value" "motor-connector" (id 1) (at 92.075 57.15 0))
-    (property "Footprint" "motor-mount:motor-mount" (id 2) (at 99.06 59.69 0)
-      (effects (font (size 1.27 1.27)) hide)
-    )
-    (property "Datasheet" "" (id 3) (at 99.06 59.69 0)
-      (effects (font (size 1.27 1.27)) hide)
-    )
+    (property "Reference" "J3" (id 0) (at 95.25 54.61 0))
+    (property "Value" "motor-connector" (id 1) (at 88.265 57.15 0))
+    (property "Footprint" "motor-mount:motor-mount" (id 2) (at 95.25 59.69 0)
+      (effects (font (size 1.27 1.27)) hide)
+    )
+    (property "Datasheet" "" (id 3) (at 95.25 59.69 0)
+      (effects (font (size 1.27 1.27)) hide)
+    )

Commit message: Remove bemf and add robins logo
Parts:
- removed D2: 2V, Diode_SMD:D_SOD-123, symbol Device:D_Zener
- removed R3: 680k, Resistor_SMD:R_0603_1608Metric, symbol Device:R
- removed R4: 120k, Resistor_SMD:R_0603_1608Metric, symbol Device:R
- C1: MPN (none) -> T491A104K035AT
- D1: MPN (none) -> SOD4007
- J1: MPN (none) -> BM04B-SRSS-TBT(LF)(SN)
- Q1: MPN (none) -> STN4NF20L
- R1: MPN (none) -> 160 0603
- R2: MPN (none) -> 100k 0603
- U1: MPN (none) -> 250X15W104MV4E
Connections:
- net BEMF is gone; now on net GND: J1.3 (Pin_3)
- net BEMF_PIN: no longer names the net of D1.2 (A), J3.1 (motor), Q1.2, Q1.T, U1.1
Other:
- note removed: "Back EMF voltage divider"
- note removed: "Vadc = Vmotor * ( 120k / ( 680k + 120k ) )"
- note removed: "Vmotor = 12V Vadc = 1.8V"

Commit message: Update val to BM04B
Parts:
- J1: value BM04B-SRSS-TBT(LF)(SN) -> BM04B
Changed lines of the file:
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@@
     (in_bom yes) (on_board yes)
     (property "Reference" "J1" (id 0) (at 49.53 60.96 0))
-    (property "Value" "BM04B-SRSS-TBT(LF)(SN)" (id 1) (at 38.735 59.055 0))
+    (property "Value" "BM04B" (id 1) (at 38.735 59.055 0))
     (property "Footprint" "Connector_JST:JST_SH_BM04B-SRSS-TB_1x04-1MP_P1.00mm_Vertical" (id 2) (at 49.53 50.8 0)
       (effects (font (size 1.27 1.27)) hide)
@@
     )
     (path "/80f92d9a-5f30-4aa7-abbe-2a03b44d3c62"
-      (reference "J1") (unit 1) (value "BM04B-SRSS-TBT(LF)(SN)") (footprint "Connector_JST:JST_SH_BM04B-SRSS-TB_1x04-1MP_P1.00mm_Vertical")
+      (reference "J1") (unit 1) (value "BM04B") (footprint "Connector_JST:JST_SH_BM04B-SRSS-TB_1x04-1MP_P1.00mm_Vertical")
     )
     (path "/487963d3-ed36-4ffe-bbc0-8af87b349b27"

Commit message: Add fiducials, fix SMD/THT, Bump rev to 4
Parts:
- added FID1, FID2: Fiducial, Fiducial:Fiducial_0.5mm_Mask1mm, symbol Mechanical:Fiducial
Changed lines of the file:
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@@
     (pin "1")
+  )
+  (symbol (lib_id "Mechanical:Fiducial") (at 23.495 21.59 0) (unit 1)
+    (in_bom yes) (on_board yes) (fields_autoplaced)
+    (property "Reference" "FID1" (id 0) (at 26.67 20.3199 0)
+      (effects (font (size 1.27 1.27)) (justify left))
+    )
+    (property "Value" "Fiducial" (id 1) (at 26.67 22.8599 0)
+      (effects (font (size 1.27 1.27)) (justify left))
+    )
+    (property "Footprint" "Fiducial:Fiducial_0.5mm_Mask1mm" (id 2) (at 23.495 21.59 0)
+      (effects (font (size 1.27 1.27)) hide)
+    )
+    (property "Datasheet" "~" (id 3) (at 23.495 21.59 0)
+      (effects (font (size 1.27 1.27)) hide)
+    )
   )
   (symbol (lib_id "Device:R") (at 133.985 81.28 0) (unit 1)
@@
     (pin "1")
   )
+  (symbol (lib_id "Mechanical:Fiducial") (at 43.815 21.59 0) (unit 1)
+    (in_bom yes) (on_board yes) (fields_autoplaced)
+    (property "Reference" "FID2" (id 0) (at 46.99 20.3199 0)
+      (effects (font (size 1.27 1.27)) (justify left))
+    )
+    (property "Value" "Fiducial" (id 1) (at 46.99 22.8599 0)
+      (effects (font (size 1.27 1.27)) (justify left))
+    )
+    (property "Footprint" "Fiducial:Fiducial_0.5mm_Mask1mm" (id 2) (at 43.815 21.59 0)
+      (effects (font (size 1.27 1.27)) hide)
+    )
+    (property "Datasheet" "~" (id 3) (at 43.815 21.59 0)
+      (effects (font (size 1.27 1.27)) hide)
+    )
+  )
   (sheet_instances
     (path "/" (page "1"))
@@
       (reference "D1") (unit 1) (value "SOD4007") (footprint "Diode_SMD:D_SOD-123F")
     )
+    (path "/9bdf1efd-4f4f-4b02-b265-4f5aa220bda6"
+      (reference "FID1") (unit 1) (value "Fiducial") (footprint "Fiducial:Fiducial_0.5mm_Mask1mm")
+    )
+    (path "/f653bc73-83d8-4dc4-8a75-da899e4932ac"
+      (reference "FID2") (unit 1) (value "Fiducial") (footprint "Fiducial:Fiducial_0.5mm_Mask1mm")
+    )
     (path "/80f92d9a-5f30-4aa7-abbe-2a03b44d3c62"

Commit message: Add 3rd fiducial
Parts:
- added FID3: Fiducial, Fiducial:Fiducial_0.5mm_Mask1mm, symbol Mechanical:Fiducial
Changed lines of the file:
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@@
   (paper "A4")
   (title_block
-    (date "2022-08-04")
+    (date "2023-01-31")
     (rev "4")
   )
@@
     (pin "1")
   )
+  (symbol (lib_id "Mechanical:Fiducial") (at 62.865 21.59 0) (unit 1)
+    (in_bom yes) (on_board yes) (fields_autoplaced)
+    (property "Reference" "FID3" (id 0) (at 66.04 20.3199 0)
+      (effects (font (size 1.27 1.27)) (justify left))
+    )
+    (property "Value" "Fiducial" (id 1) (at 66.04 22.8599 0)
+      (effects (font (size 1.27 1.27)) (justify left))
+    )
+    (property "Footprint" "Fiducial:Fiducial_0.5mm_Mask1mm" (id 2) (at 62.865 21.59 0)
+      (effects (font (size 1.27 1.27)) hide)
+    )
+    (property "Datasheet" "~" (id 3) (at 62.865 21.59 0)
+      (effects (font (size 1.27 1.27)) hide)
+    )
+  )
   (symbol (lib_id "power:GND") (at 105.41 62.865 0) (unit 1)
     (in_bom yes) (on_board yes)
@@
       (reference "FID2") (unit 1) (value "Fiducial") (footprint "Fiducial:Fiducial_0.5mm_Mask1mm")
     )
+    (path "/bf17c75a-8397-441d-98f1-eca78915375f"
+      (reference "FID3") (unit 1) (value "Fiducial") (footprint "Fiducial:Fiducial_0.5mm_Mask1mm")
+    )
     (path "/80f92d9a-5f30-4aa7-abbe-2a03b44d3c62"

Commit message: Add kikit tabs
Parts:
- added T? (x2): Tab, kikit:Tab, symbol kikit:Tab
Changed lines of the file:
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@@
     (pin "1")
+  )
+  (symbol (lib_id "kikit:Tab") (at 199.39 45.085 0) (unit 1)
+    (in_bom no) (on_board yes) (fields_autoplaced)
+    (property "Reference" "T?" (id 0) (at 204.47 43.1799 0)
+      (effects (font (size 1.27 1.27)) (justify left))
+    )
+    (property "Value" "Tab" (id 1) (at 204.47 45.7199 0)
+      (effects (font (size 1.27 1.27)) (justify left))
+    )
+    (property "Footprint" "kikit:Tab" (id 2) (at 199.39 45.085 0)
+      (effects (font (size 1.27 1.27)) hide)
+    )
+    (property "Datasheet" "" (id 3) (at 199.39 45.085 0)
+      (effects (font (size 1.27 1.27)) hide)
+    )
   )
   (symbol (lib_id "power:GND") (at 142.875 86.36 0) (unit 1)
@@
     )
     (pin "1")
+  )
+  (symbol (lib_id "kikit:Tab") (at 216.535 45.085 0) (unit 1)
+    (in_bom no) (on_board yes) (fields_autoplaced)
+    (property "Reference" "T?" (id 0) (at 221.615 43.1799 0)
+      (effects (font (size 1.27 1.27)) (justify left))
+    )
+    (property "Value" "Tab" (id 1) (at 221.615 45.7199 0)
+      (effects (font (size 1.27 1.27)) (justify left))
+    )
+    (property "Footprint" "kikit:Tab" (id 2) (at 216.535 45.085 0)
+      (effects (font (size 1.27 1.27)) hide)
+    )
+    (property "Datasheet" "" (id 3) (at 216.535 45.085 0)
+      (effects (font (size 1.27 1.27)) hide)
+    )
   )
   (symbol (lib_id "power:+12V") (at 61.595 43.815 0) (unit 1)
@@
       (reference "R2") (unit 1) (value "100k") (footprint "Resistor_SMD:R_0603_1608Metric")
     )
+    (path "/7955651d-e9d7-4ddf-897b-611f0100c74b"
+      (reference "T?") (unit 1) (value "Tab") (footprint "kikit:Tab")
+    )
+    (path "/a8816ebb-c11f-49cc-a261-ae6bea964554"
+      (reference "T?") (unit 1) (value "Tab") (footprint "kikit:Tab")
+    )
     (path "/c99d9ee8-b4c6-4374-bb5b-0809ce253ad3"
