File: pixel-pump-motor-board.kicad_sch (KiCad schematic)
At the start: 18 parts, among them J1 BM04B, J11 Motor Chassis GND, J2 motor-connector, J3 motor-connector, J5 Motor Chassis GND, J7 Motor Chassis GND, J8 Motor Chassis GND, Q1 STN4NF20L, U1 250X15W104MV4E

Commit message: Add tabs to schematics
Parts:
- gave numbers to parts that had none: 2
Changed lines of the file:
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@@
   (symbol (lib_id "kikit:Tab") (at 199.39 45.085 0) (unit 1)
     (in_bom no) (on_board yes) (fields_autoplaced)
-    (property "Reference" "T?" (id 0) (at 204.47 43.1799 0)
+    (property "Reference" "T1" (id 0) (at 204.47 43.1799 0)
       (effects (font (size 1.27 1.27)) (justify left))
     )
@@
   (symbol (lib_id "kikit:Tab") (at 216.535 45.085 0) (unit 1)
     (in_bom no) (on_board yes) (fields_autoplaced)
-    (property "Reference" "T?" (id 0) (at 221.615 43.1799 0)
+    (property "Reference" "T2" (id 0) (at 221.615 43.1799 0)
       (effects (font (size 1.27 1.27)) (justify left))
     )
@@
     )
     (path "/7955651d-e9d7-4ddf-897b-611f0100c74b"
-      (reference "T?") (unit 1) (value "Tab") (footprint "kikit:Tab")
+      (reference "T1") (unit 1) (value "Tab") (footprint "kikit:Tab")
     )
     (path "/a8816ebb-c11f-49cc-a261-ae6bea964554"
-      (reference "T?") (unit 1) (value "Tab") (footprint "kikit:Tab")
+      (reference "T2") (unit 1) (value "Tab") (footprint "kikit:Tab")
     )
     (path "/c99d9ee8-b4c6-4374-bb5b-0809ce253ad3"

Commit message: Fixed footprints
Parts:
- C1: value 100n 25V -> 100N 25V
- J1: value BM04B -> BM04B-SRSS-TBT
- R1: value 160 -> 160R
- R2: value 100k -> 100K
Other:
- moved on the sheet: R1
Changed lines of the file:
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@@
-    (stroke (width 0) (type solid) (color 0 0 0 0))
-  )
-  (wire (pts (xy 126.365 74.93) (xy 126.365 78.74))
     (stroke (width 0) (type solid) (color 0 0 0 0))
   )
@@
     (stroke (width 0) (type solid) (color 0 0 0 0))
   )
-  (wire (pts (xy 126.365 74.93) (xy 133.985 74.93))
+  (wire (pts (xy 123.825 74.93) (xy 133.985 74.93))
     (stroke (width 0) (type solid) (color 0 0 0 0))
   )
@@
     (stroke (width 0) (type solid) (color 0 0 0 0))
   )
+  (wire (pts (xy 123.825 74.93) (xy 123.825 78.74))
+    (stroke (width 0) (type default) (color 0 0 0 0))
+  )
   (wire (pts (xy 156.845 130.81) (xy 156.845 137.16))
     (stroke (width 0) (type solid) (color 0 0 0 0))
@@
     (stroke (width 0) (type solid) (color 0 0 0 0))
   )
-  (wire (pts (xy 126.365 86.36) (xy 126.365 88.9))
+  (wire (pts (xy 123.825 86.36) (xy 123.825 88.9))
     (stroke (width 0) (type solid) (color 0 0 0 0))
   )
@@
     )
   )
-  (global_label "PWM" (shape input) (at 126.365 88.9 270)
+  (global_label "PWM" (shape input) (at 123.825 88.9 270)
     (effects (font (size 1.27 1.27)) (justify right))
-    (property "Intersheet References" "${INTERSHEET_REFS}" (id 0) (at 57.785 314.96 0)
+    (property "Intersheet References" "${INTERSHEET_REFS}" (id 0) (at 55.245 314.96 0)
       (effects (font (size 1.27 1.27)) hide)
     )
@@
   (symbol (lib_id "Device:C_Polarized") (at 158.115 55.88 0) (unit 1)
     (in_bom yes) (on_board yes) (fields_autoplaced)
-    (property "Reference" "C1" (id 0) (at 161.925 55.2449 0)
-      (effects (font (size 1.27 1.27)) (justify left))
-    )
-    (property "Value" "100n 25V" (id 1) (at 161.925 57.7849 0)
+    (property "Reference" "C1" (id 0) (at 161.29 53.7209 0)
+      (effects (font (size 1.27 1.27)) (justify left))
+    )
+    (property "Value" "100N 25V" (id 1) (at 161.29 56.2609 0)
       (effects (font (size 1.27 1.27)) (justify left))
     )
@@
     (in_bom yes) (on_board yes)
     (property "Reference" "J1" (id 0) (at 49.53 60.96 0))
-    (property "Value" "BM04B" (id 1) (at 38.735 59.055 0))
+    (property "Value" "BM04B-SRSS-TBT" (id 1) (at 38.735 59.055 0))
     (property "Footprint" "Connector_JST:JST_SH_BM04B-SRSS-TB_1x04-1MP_P1.00mm_Vertical" (id 2) (at 49.53 50.8 0)
       (effects (font (size 1.27 1.27)) hide)
@@
       (effects (font (size 1.27 1.27)) (justify left))
     )
-    (property "Value" "100k" (id 1) (at 135.763 82.423 0)
+    (property "Value" "100K" (id 1) (at 135.763 82.423 0)
       (effects (font (size 1.27 1.27)) (justify left))
     )
@@
     (pin "4")
   )
-  (symbol (lib_id "Device:R") (at 126.365 82.55 0) (unit 1)
-    (in_bom yes) (on_board yes)
-    (property "Reference" "R1" (id 0) (at 128.143 81.3816 0)
-      (effects (font (size 1.27 1.27)) (justify left))
-    )
-    (property "Value" "160" (id 1) (at 128.143 83.693 0)
-      (effects (font (size 1.27 1.27)) (justify left))
-    )
-    (property "Footprint" "Resistor_SMD:R_0603_1608Metric" (id 2) (at 124.587 82.55 90)
-      (effects (font (size 1.27 1.27)) hide)
-    )
-    (property "Datasheet" "~" (id 3) (at 126.365 82.55 0)
-      (effects (font (size 1.27 1.27)) hide)
-    )
-    (property "MPN" "160 0603" (id 4) (at 126.365 82.55 0)
+  (symbol (lib_id "Device:R") (at 123.825 82.55 0) (unit 1)
+    (in_bom yes) (on_board yes)
+    (property "Reference" "R1" (id 0) (at 125.603 81.3816 0)
+      (effects (font (size 1.27 1.27)) (justify left))
+    )
+    (property "Value" "160R" (id 1) (at 125.603 83.693 0)
+      (effects (font (size 1.27 1.27)) (justify left))
+    )
+    (property "Footprint" "Resistor_SMD:R_0603_1608Metric" (id 2) (at 122.047 82.55 90)
+      (effects (font (size 1.27 1.27)) hide)
+    )
+    (property "Datasheet" "~" (id 3) (at 123.825 82.55 0)
+      (effects (font (size 1.27 1.27)) hide)
+    )
+    (property "MPN" "160 0603" (id 4) (at 123.825 82.55 0)
       (effects (font (size 1.27 1.27)) hide)
     )
@@
     )
     (path "/1f7a19e5-e285-4bb1-bf4e-7d1ea9a40a35"
-      (reference "C1") (unit 1) (value "100n 25V") (footprint "Capacitor_Tantalum_SMD:CP_EIA-3216-18_Kemet-A")
+      (reference "C1") (unit 1) (value "100N 25V") (footprint "Capacitor_Tantalum_SMD:CP_EIA-3216-18_Kemet-A")
     )
     (path "/0e0e6608-be18-4a36-8a5f-fc659e496bef"
@@
     )
     (path "/80f92d9a-5f30-4aa7-abbe-2a03b44d3c62"
-      (reference "J1") (unit 1) (value "BM04B") (footprint "Connector_JST:JST_SH_BM04B-SRSS-TB_1x04-1MP_P1.00mm_Vertical")
+      (reference "J1") (unit 1) (value "BM04B-SRSS-TBT") (footprint "Connector_JST:JST_SH_BM04B-SRSS-TB_1x04-1MP_P1.00mm_Vertical")
     )
     (path "/487963d3-ed36-4ffe-bbc0-8af87b349b27"
@@
     )
     (path "/d3a2a931-a2c2-464e-a9ce-2f97b6278923"
-      (reference "R1") (unit 1) (value "160") (footprint "Resistor_SMD:R_0603_1608Metric")
+      (reference "R1") (unit 1) (value "160R") (footprint "Resistor_SMD:R_0603_1608Metric")
     )
     (path "/9d39777c-df04-4406-bea8-e238b0cc7a3d"
-      (reference "R2") (unit 1) (value "100k") (footprint "Resistor_SMD:R_0603_1608Metric")
+      (reference "R2") (unit 1) (value "100K") (footprint "Resistor_SMD:R_0603_1608Metric")
     )
     (path "/7955651d-e9d7-4ddf-897b-611f0100c74b"

Commit message: Add BM04B footprint
Parts:
- J1: footprint Connector_JST:JST_SH_BM04B-SRSS-TB_1x04-1MP_P1.00mm_Vertical -> BM04B-SRSS-TBT:BM04B-SRSS-TBT
Changed lines of the file:
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@@
     (property "Reference" "J1" (id 0) (at 49.53 60.96 0))
     (property "Value" "BM04B-SRSS-TBT" (id 1) (at 38.735 59.055 0))
-    (property "Footprint" "Connector_JST:JST_SH_BM04B-SRSS-TB_1x04-1MP_P1.00mm_Vertical" (id 2) (at 49.53 50.8 0)
+    (property "Footprint" "BM04B-SRSS-TBT:BM04B-SRSS-TBT" (id 2) (at 49.53 50.8 0)
       (effects (font (size 1.27 1.27)) hide)
     )
@@
     )
     (path "/80f92d9a-5f30-4aa7-abbe-2a03b44d3c62"
-      (reference "J1") (unit 1) (value "BM04B-SRSS-TBT") (footprint "Connector_JST:JST_SH_BM04B-SRSS-TB_1x04-1MP_P1.00mm_Vertical")
+      (reference "J1") (unit 1) (value "BM04B-SRSS-TBT") (footprint "BM04B-SRSS-TBT:BM04B-SRSS-TBT")
     )
     (path "/487963d3-ed36-4ffe-bbc0-8af87b349b27"
